File: Circuito/Fonte12V.brd (EAGLE design)
At the start: 100 x 80 mm, 9 parts, among them T1 2N706

Commit message: README
Parts:
- added LED: TLLR4400, led:LED3MM
- added R1: 1.1k, rcl:0207/10
- moved D1 23.6 mm to (62.2, 53.3)
- moved R4 22.2 mm to (62.2, 62.2)
- moved T1 15.1 mm to (31.2, 53.3)
- moved R2 7.41 mm to (41.9, 41.9)
- moved B1 7.41 mm to (21.6, 66.0)
- moved SAIDA 7.18 mm to (3.81, 54.6), turned to 90 degrees
- moved C1 6.84 mm to (33.0, 61.0), turned to 270 degrees
- moved R3 2.84 mm to (19.1, 48.3)
- moved ENTRADA 2.54 mm to (10.2, 76.2)
Connections:
- new net N$9: LED.A, R1.1
- net N$1: now also R1.2
- net N$2: now also LED.K
Routing:
- net N$2: track 126.7 -> 69.2 mm
- net N$1: track 32.3 -> 86.2 mm
- net N$6: track 8.89 -> 31.7 mm
- net N$5: track 7.70 -> 15.4 mm
- net N$4: track 21.6 -> 14.1 mm
- net N$3: track 22.1 -> 15.9 mm
- net N$9: track 0.00 -> 5.08 mm
- net N$8: track 20.6 -> 16.9 mm
- net N$7: track 35.6 -> 35.0 mm
