File: Circuito/Fonte12V.sch (EAGLE design)
At the start: 9 parts, among them T1 2N706

Commit message: README
Parts:
- added LED: TLLR4400, led:TLLR4400
- added R1: 1.1k, rcl:R-EU_0207/10
Connections:
- new net N$9: LED.A, R1.1
- net N$1: now also R1.2
- net N$2: now also LED.C
Changed lines of the file:
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@@
 <part name="R3" library="rcl" library_urn="urn:adsk.eagle:library:334" deviceset="R-EU_" device="0207/10" package3d_urn="urn:adsk.eagle:package:23491/2" value="2.2k"/>
 <part name="R4" library="rcl" library_urn="urn:adsk.eagle:library:334" deviceset="R-EU_" device="0207/10" package3d_urn="urn:adsk.eagle:package:23491/2" value="330"/>
+<part name="R1" library="rcl" library_urn="urn:adsk.eagle:library:334" deviceset="R-EU_" device="0207/10" package3d_urn="urn:adsk.eagle:package:23491/2" value="1.1k"/>
+<part name="LED" library="led" library_urn="urn:adsk.eagle:library:259" deviceset="TLLR4400" device="" package3d_urn="urn:adsk.eagle:package:15797/1"/>
 </parts>
 <sheets>
@@
 </plain>
 <instances>
-<instance part="T1" gate="G$1" x="48.26" y="2.54" smashed="yes">
-<attribute name="NAME" x="38.1" y="10.16" size="1.778" layer="95"/>
-<attribute name="VALUE" x="38.1" y="7.62" size="1.778" layer="96"/>
-</instance>
+<instance part="T1" gate="G$1" x="48.26" y="2.54" smashed="yes"/>
 <instance part="R2" gate="G$1" x="40.64" y="2.54" smashed="yes">
-<attribute name="NAME" x="34.671" y="-1.27" size="1.778" layer="95" rot="R90"/>
 <attribute name="VALUE" x="36.83" y="-1.27" size="1.778" layer="96" rot="R90"/>
 </instance>
@@
 <attribute name="NAME" x="-5.08" y="-5.08" size="1.778" layer="95" rot="R180"/>
 </instance>
-<instance part="C1" gate="G$1" x="20.32" y="-2.54" smashed="yes">
-<attribute name="NAME" x="21.463" y="-2.0574" size="1.778" layer="95"/>
-<attribute name="VALUE" x="21.463" y="-7.1374" size="1.778" layer="96"/>
+<instance part="C1" gate="G$1" x="17.78" y="0" smashed="yes">
+<attribute name="VALUE" x="18.923" y="-4.5974" size="1.778" layer="96"/>
 </instance>
 <instance part="ENTRADA" gate="G$1" x="-43.18" y="-2.54" smashed="yes" rot="R180">
@@
 </instance>
 <instance part="R3" gate="G$1" x="40.64" y="-10.16" smashed="yes" rot="R90">
-<attribute name="NAME" x="39.1414" y="-13.97" size="1.778" layer="95" rot="R90"/>
 <attribute name="VALUE" x="43.942" y="-13.97" size="1.778" layer="96" rot="R90"/>
 </instance>
 <instance part="R4" gate="G$1" x="33.02" y="12.7" smashed="yes" rot="R90">
-<attribute name="NAME" x="31.5214" y="8.89" size="1.778" layer="95" rot="R90"/>
 <attribute name="VALUE" x="36.322" y="8.89" size="1.778" layer="96" rot="R90"/>
+</instance>
+<instance part="R1" gate="G$1" x="25.4" y="7.62" smashed="yes" rot="R90">
+<attribute name="VALUE" x="28.702" y="3.81" size="1.778" layer="96" rot="R90"/>
+</instance>
+<instance part="LED" gate="G$1" x="25.4" y="-15.24" smashed="yes">
+<attribute name="NAME" x="28.956" y="-19.812" size="1.778" layer="95" rot="R90"/>
 </instance>
 </instances>
@@
 <net name="N$1" class="0">
 <segment>
-<wire x1="20.32" y1="0" x2="20.32" y2="17.78" width="0.1524" layer="91"/>
-<wire x1="20.32" y1="17.78" x2="33.02" y2="17.78" width="0.1524" layer="91"/>
+<wire x1="17.78" y1="2.54" x2="17.78" y2="17.78" width="0.1524" layer="91"/>
+<wire x1="17.78" y1="17.78" x2="25.4" y2="17.78" width="0.1524" layer="91"/>
 <pinref part="T1" gate="G$1" pin="C"/>
+<wire x1="25.4" y1="17.78" x2="33.02" y2="17.78" width="0.1524" layer="91"/>
 <wire x1="33.02" y1="17.78" x2="50.8" y2="17.78" width="0.1524" layer="91"/>
 <wire x1="50.8" y1="17.78" x2="50.8" y2="7.62" width="0.1524" layer="91"/>
-<wire x1="20.32" y1="17.78" x2="-12.7" y2="17.78" width="0.1524" layer="91"/>
-<junction x="20.32" y="17.78"/>
+<wire x1="17.78" y1="17.78" x2="-12.7" y2="17.78" width="0.1524" layer="91"/>
+<junction x="17.78" y="17.78"/>
 <wire x1="-12.7" y1="17.78" x2="-12.7" y2="-2.54" width="0.1524" layer="91"/>
 <pinref part="C1" gate="G$1" pin="+"/>
@@
 <pinref part="R4" gate="G$1" pin="2"/>
 <junction x="33.02" y="17.78"/>
+<pinref part="R1" gate="G$1" pin="2"/>
+<wire x1="25.4" y1="17.78" x2="25.4" y2="12.7" width="0.1524" layer="91"/>
+<junction x="25.4" y="17.78"/>
 </segment>
 </net>
@@
 <wire x1="40.64" y1="-15.24" x2="40.64" y2="-22.86" width="0.1524" layer="91"/>
 <wire x1="40.64" y1="-22.86" x2="33.02" y2="-22.86" width="0.1524" layer="91"/>
-<wire x1="33.02" y1="-22.86" x2="20.32" y2="-22.86" width="0.1524" layer="91"/>
-<wire x1="20.32" y1="-22.86" x2="12.7" y2="-22.86" width="0.1524" layer="91"/>
+<wire x1="33.02" y1="-22.86" x2="25.4" y2="-22.86" width="0.1524" layer="91"/>
+<wire x1="25.4" y1="-22.86" x2="17.78" y2="-22.86" width="0.1524" layer="91"/>
+<wire x1="17.78" y1="-22.86" x2="12.7" y2="-22.86" width="0.1524" layer="91"/>
 <wire x1="12.7" y1="-22.86" x2="12.7" y2="-2.54" width="0.1524" layer="91"/>
-<wire x1="20.32" y1="-7.62" x2="20.32" y2="-22.86" width="0.1524" layer="91"/>
-<junction x="20.32" y="-22.86"/>
+<wire x1="17.78" y1="-5.08" x2="17.78" y2="-22.86" width="0.1524" layer="91"/>
+<junction x="17.78" y="-22.86"/>
 <pinref part="C1" gate="G$1" pin="-"/>
 <pinref part="B1" gate="1" pin="-"/>
@@
 <junction x="33.02" y="-22.86"/>
 <pinref part="R3" gate="G$1" pin="1"/>
+<pinref part="LED" gate="G$1" pin="C"/>
+<wire x1="25.4" y1="-20.32" x2="25.4" y2="-22.86" width="0.1524" layer="91"/>
+<junction x="25.4" y="-22.86"/>
 </segment>
 </net>
@@
 </segment>
 </net>
+<net name="N$9" class="0">
+<segment>
+<pinref part="R1" gate="G$1" pin="1"/>
+<wire x1="25.4" y1="2.54" x2="25.4" y2="-12.7" width="0.1524" layer="91"/>
+<pinref part="LED" gate="G$1" pin="A"/>
+</segment>
+</net>
